File: MainBoard/Power.kicad_sch (KiCad schematic)
At the start: 121 parts, among them J301 Delphi_Sicma_24, J302 USB_A, J404 USB_B_Mini, K301 G6K-2F-Y DC12, Q301 S8550, Q302 S8550, Q303 S8550, Q304 S8550, Q305 S8550, Q306 S8550, Q307 S8550, Q308 S8550, Q309 SI2302-TP, Q310 SI2302-TP, Q311 SI2302-TP, Q312 S8550, Q313 S8550, Q314 S8550, Q315 S8550, Q316 S8550, Q317 S8550, Q318 S8550, Q319 SI2302-TP, Q320 SI2302-TP, Q321 SI2302-TP, Q322 SI2301CDS-T1-GE3, U301 SCT2650STER, U302 USBLC6-2SC6, U303 USBLC6-2SC6, U402 SY8088IAAC, U403 SY8088IAAC, U405 SN65HVD230

Commit message: Submit for fab rev 2
Signed-off-by: Connor Rigby <connorr@hey.com>
Parts:
- removed C307: 220uF 16V, Capacitor_SMD:CP_Elec_10x10, symbol Device:C_Polarized
- removed Q301, Q302, Q303, Q304, Q305, Q306, Q307, Q313, Q314, Q315, Q316, Q317, Q318: S8550, Package_TO_SOT_SMD:SOT-23, symbol Transistor_BJT:BC850
- removed Q322: SI2301CDS-T1-GE3, Package_TO_SOT_SMD:SOT-23, symbol Transistor_FET:Si2319CDS
- removed R402: 1k, Resistor_SMD:R_0402_1005Metric, symbol Device:R
- added C316, C318: 10uF, Capacitor_SMD:C_0603_1608Metric, symbol Device:C
- added C317, C319, C321, C323, C325, C327: 100nf, Capacitor_SMD:C_0402_1005Metric, symbol Device:C_Small
- added Q301, Q304, Q307: AO3419, Package_TO_SOT_SMD:SOT-23W, symbol Device:Q_PMOS_GSD
- added Q302, Q303, Q305, Q306: SI2302-TP, Package_TO_SOT_SMD:SOT-23, symbol Device:Q_NMOS_GSD
- added TP301: +5V, TestPoint:TestPoint_Pad_D1.0mm, symbol Connector:TestPoint
- added TP302, TP304: gnd, TestPoint:TestPoint_Pad_D1.0mm, symbol Connector:TestPoint
- added TP303: +3.3V, TestPoint:TestPoint_Pad_D1.0mm, symbol Connector:TestPoint
- added U304, U305, U306, U307, U308, U309: MCP1416T-E/OT, Package_TO_SOT_SMD:SOT-23-5, symbol Driver_FET:MCP1416
- Q308, Q312: value S8550 -> MMBT5551; LCSC C105432 -> C2145; MPN S8550 -> MMBT5551
- R305: now left out of the parts list
- R306, R328: value 100k 1% -> 22R; LCSC C25741 -> C25092; MPN 0402WGF1003TCE -> 0402WGF220JTCE
- R316, R317, R318, R330: value 100k 1% -> 1k; LCSC C25741 -> C11702; MPN 0402WGF1003TCE -> 0402WGF1001TCE
- R321, R322, R331, R333, R334: value 1k -> 100k 1%; LCSC C11702 -> C25741; MPN 0402WGF1001TCE -> 0402WGF1003TCE
- R323, R324: value 1k -> 22R; LCSC C11702 -> C25092; MPN 0402WGF1001TCE -> 0402WGF220JTCE
Connections:
- net +3V3: now also D409.2 (A), TP303.1; no longer D409.1 (K)
- net +5V: now also D408.2 (A), R322.2, R333.2, Q301.2 (S), Q304.2 (S), Q307.2 (S); no longer D408.1 (K)
- net GND: now also R321.2, R331.2, R334.2, C316.2, C317.2, C318.2, C319.2, C321.2, C323.2, C325.2, C327.2, Q302.2 (S), Q303.2 (S), Q305.2 (S), Q306.2 (S), TP302.1, TP304.1, U304.4 (GND), U305.4 (GND), U306.4 (GND), U307.4 (GND), U308.4 (GND), U309.4 (GND); no longer R306.2, R316.2, R317.2, R318.2, R328.2, R330.2
- net RELAY_SW: now also R320.1, R321.1
- net RGB1_OUT: now also C316.1, C317.1, C319.1, C321.1, U304.2 (Vdd), U305.2 (Vdd), U306.2 (Vdd); no longer R319.1, R320.1, R321.1, R322.1, R323.1, R324.1
- net RGB2_OUT: now also C318.1, C323.1, C325.1, C327.1, U307.2 (Vdd), U308.2 (Vdd), U309.2 (Vdd); no longer R301.1, R302.1, R331.1, R332.1, R333.1, R334.1
- net VIN: no longer D305.1 (K), K301.1
- net at C308.1, C309.1, C310.1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: now also TP301.1
- net at R303.1: now also R334.1, Q307.1 (G)
- net at J302.1 (VBUS), U302.5 (VBUS): now also Q307.3 (D)
- net at R436.2: now also U304.3 (IN); no longer R316.1
- net at R306.1: now also Q301.3 (D)
- net at D305.2 (A), K301.8: now also R323.2, R324.2
- net RGB2_B_G: now reaches R319.2
- net RGB2_B_G: now also Q321.1 (G)
- net RGB1_R_G: now reaches Q309.1 (G)
- net RGB1_R_G: now also R301.2; no longer R322.2
- net at R427.2: now also D408.1 (K); no longer D408.2 (A)
- net at R430.1: now also U309.3 (IN); no longer R330.1
- net at R332.2: now also Q306.1 (G)
- net at R317.1: now also U307.5 (OUT); no longer R435.2
- net at R320.2: now also Q302.1 (G)
- net RGB1_B_G: now reaches Q311.1 (G)
- net RGB1_B_G: now also R316.2; no longer R324.2
- net RGB1_G_G: now reaches R302.2
- net RGB1_G_G: now also Q310.1 (G); no longer Q319.1 (G)
- net RGB2_G_G: now reaches Q320.1 (G)
- net RGB2_G_G: now also R318.2; no longer R333.2
- net at R434.1: now also U308.3 (IN); no longer R329.1
- net at R428.2: now also D409.1 (K); no longer D409.2 (A)
- net at R411.1: now also U306.3 (IN); no longer R318.1
- net at R408.1: now also U307.3 (IN); no longer R328.1
- new net: R435.2, U305.3 (IN)
- new net: R302.1, U305.5 (OUT)
- new net: Q305.1 (G), R330.2
- new net: Q302.3 (D), Q303.1 (G), Q304.1 (G), R322.1
- new net: R301.1, U304.5 (OUT)
- new net: Q301.1 (G), Q306.3 (D), R333.1
- new net: D305.1 (K), K301.1, R306.2, R328.2
- new net: R319.1, U309.5 (OUT)
- new net: Q304.3 (D), R323.1
- new net: Q303.3 (D), R324.1
- new net: Q305.3 (D), R328.1
- new net: R318.1, U308.5 (OUT)
- new net: R316.1, U306.5 (OUT)
- new net RELAY_COIL_GND: R329.1, R330.1
- new net RELAY_COIL_VDC: R331.1, R332.1
- new net RGB2_R_G: Q319.1 (G), R317.2
Other:
- moved on the sheet: C301, C302, C303, C304, C305, C306, C308, C309, C310, C311, C313, C314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

Commit message: Submit for production
Signed-off-by: Connor Rigby <connorr@hey.com>
Parts:
- removed C301: 1uF, Resistor_SMD:R_0402_1005Metric, symbol Device:C_Small
- removed C305: 22pF, Capacitor_SMD:C_0402_1005Metric, symbol Device:C
- removed C306: 3.3nF, Capacitor_SMD:C_0402_1005Metric, symbol Device:C
- removed C308: 10uF, Capacitor_SMD:C_0603_1608Metric, symbol Device:C
- removed C309: 220nF, Capacitor_SMD:C_0603_1608Metric, symbol Device:C
- removed C310: 68pF, Capacitor_SMD:C_0603_1608Metric, symbol Device:C
- removed FB302: 450mΩ ±25% 600Ω@100MHz, Inductor_SMD:L_0603_1608Metric, symbol Device:FerriteBead
- removed L301: 8.2uH 3.7A, Inductor_LCSC:IND-SMD_L7.0-W6.6_FXL0630, symbol Device:L
- removed L302: 2.2uH, Inductor_SMD:L_0603_1608Metric, symbol Device:L
- removed Q308, Q312: MMBT5551, Package_TO_SOT_SMD:SOT-23, symbol Transistor_BJT:BC850
- removed R304, R305: 0R, Resistor_SMD:R_0402_1005Metric, symbol Device:R_Small
- removed R309, R310, R314: 100k 1%, Resistor_SMD:R_0402_1005Metric, symbol Device:R
- removed R313: 33k 1%, Resistor_SMD:R_0402_1005Metric, symbol Device:R
- removed R315: 18.7k 1%, Resistor_SMD:R_0402_1005Metric, symbol Device:R
- removed R446: 1k, Resistor_SMD:R_0402_1005Metric, symbol Device:R
- removed U301: SCT2650STER, Package_SO:HSOP-8-1EP_3.9x4.9mm_P1.27mm_EP2.41x3.1mm, symbol LCSC_Regulator:SCT2650STER
- removed U302, U303: USBLC6-2SC6, Package_TO_SOT_SMD:SOT-23-6, symbol Power_Protection:USBLC6-2SC6
- added C307, C320: 10uF 16V, Capacitor_Tantalum_SMD:CP_EIA-3216-18_Kemet-A, symbol Device:C_Polarized
- added D301, D302, D303, D307, D308, D309, D310, D311, D312: LED, LED_SMD:LED_0402_1005Metric, symbol Device:LED
- added D313: NSR0320MW2T1G, Diode_SMD:D_SOD-323, symbol Device:D
- added L303: 4.7uH, easyeda2kicad:IND-SMD_L7.3-W7.3, symbol Device:L
- added R335, R336, R337, R338, R339, R340, R341, R342, R343: 1k, Resistor_SMD:R_0402_1005Metric, symbol Device:R_Small
- added R344, R345, R346: 100k 1%, Resistor_SMD:R_0402_1005Metric, symbol Device:R
- added R347: 10k, Resistor_SMD:R_0402_1005Metric, symbol Device:R_Small
- added R348: 3.3k, Resistor_SMD:R_0402_1005Metric, symbol Device:R_Small
- added U302, U303: SRV05-4, Package_TO_SOT_SMD:SOT-23-6, symbol Power_Protection:SRV05-4
- added U310: TPS5430DDA, Package_SO:TI_SO-PowerPAD-8_ThermalVias, symbol Regulator_Switching:TPS5430DDA
- C316, C318, C403, C404, C407, C408, C409, C412: LCSC C466780 -> C19702; MPN C0603X5R106M100NT -> CL10A106KP8NNNC
- J301: MPN (none) -> Delphi_Sicma_24; now not fitted; now left out of the parts list
- K301: value G6K-2F-Y DC12 -> G6K-2F-Y-TR DC3; LCSC C397194 -> C2153097; MPN G6K-2F-Y DC12 -> G6K-2F-Y-TR DC3
- R307, R311: footprint Resistor_SMD:R_0603_1608Metric -> Resistor_SMD:R_0402_1005Metric; LCSC C25804 -> C25744; MPN 0603WAF1002T5E -> 0402WGF1002TCE
- R308, R312: value 2.2k -> 3.9k; footprint Resistor_SMD:R_0603_1608Metric -> Resistor_SMD:R_0402_1005Metric; LCSC C4190 -> C51721; MPN 0603WAF2201T5E -> 0402WGF3901TCE; Resistance 2.2k -> 3.9k
- R326, R327: value 1k -> 100k 1%; LCSC C11702 -> C25741; MPN 0402WGF1001TCE -> 0402WGF1003TCE
- U304, U305, U306, U307, U308, U309: MPN (none) -> MCP1416T-E/OT
Connections:
- net +5V: now also C311.1, C313.1, C314.1, TP301.1, D301.2 (A), D302.2 (A), D303.2 (A), D307.2 (A), D308.2 (A), D309.2 (A), D310.2 (A), D311.2 (A), D312.2 (A), L303.2, R347.1; no longer R326.1, R327.1
- net GND: now also R325.1, R326.1, R327.1, C307.2, C320.2, R344.1, R345.1, R346.1, R348.2, U302.2 (VN), U303.2 (VN), U310.6 (GND), U310.9 (GNDPAD); no longer R325.2
- net LEDC: now also D313.2 (A)
- net LEDC_OUT: now also D313.1 (K); no longer R327.2
- net PWM_B1: now also R337.1
- net PWM_B2: now also R340.1
- net PWM_G1: now also R336.1
- net PWM_G2: now also R339.1
- net PWM_R1: now also R335.1
- net PWM_R2: now also R338.1
- net RELAY_COIL_GND: now also R342.1
- net RELAY_COIL_VDC: now also R343.1
- net RELAY_SW: now also R341.1
- net RGB1_OUT: now also C320.1
- net RGB2_OUT: now also C307.1
- net USB0_DN: now also J404.2 (D-), U303.1 (IO1), U303.6 (IO4)
- net USB0_DP: now also J404.3 (D+), U303.3 (IO2), U303.4 (IO3)
- net USB1_DN: now also J302.2 (D-), U302.1 (IO1), U302.6 (IO4)
- net USB1_DP: now also J302.3 (D+), U302.3 (IO2), U302.4 (IO3)
- net VBUS: now also U303.5 (VP)
- net at R408.1, U307.3 (IN): now also R346.2
- net at J302.1 (VBUS), Q307.3 (D): now also U302.5 (VP)
- net at R435.2, U305.3 (IN): now also R326.2
- net at R436.2, U304.3 (IN): now also R325.2
- net at C302.1, C303.1, D304.1 (K): now also U310.5 (EN), U310.7 (VIN)
- net at R434.1, U308.3 (IN): now also R345.2
- net at R411.1, U306.3 (IN): now also R327.2
- net at R430.1, U309.3 (IN): now also R344.2
- net at J302.5 (Shield): now also J302.6 (Shield)
- net BOOT: now reaches C304.1
- net BOOT: now also U310.1 (BOOT)
- net SW renamed PH
- net PH: now also L303.1, U310.8 (PH)
- new net: D301.1 (K), R335.2
- new net: D303.1 (K), R337.2
- new net: D308.1 (K), R339.2
- new net: D312.1 (K), R343.2
- new net: D307.1 (K), R338.2
- new net: D311.1 (K), R342.2
- new net: D310.1 (K), R341.2
- new net: D309.1 (K), R340.2
- new net: D302.1 (K), R336.2
- new net VSENSE: R347.2, R348.1, U310.4 (VSENSE)
Other:
- moved on the sheet: C304, C311, C313, C314, Q307, R303, R334, R411, R435, R436, TP302
