File: MainBoard/RL-SM02BD-8723BS.kicad_sch (KiCad schematic)
At the start: 20 parts, among them U401 RTL8723BS(ComboModule)

Commit message: Submit for fab rev 2
Signed-off-by: Connor Rigby <connorr@hey.com>
Parts:
- removed C401: 1uF, Resistor_SMD:R_0402_1005Metric, symbol Device:C_Small
- removed C417: 100nf, Capacitor_SMD:C_0402_1005Metric, symbol Device:C_Small
- removed R459: 0R, Resistor_SMD:R_0402_1005Metric, symbol Device:R_Small
- removed U401: RTL8723BS(ComboModule), Module_WiFi_BT:RL-SM02BD(RTL8723BS), symbol Module_WiFi_BT:RTL8723BS(ComboModule)
- added C402, C414: 22pF, Capacitor_SMD:C_0402_1005Metric, symbol Device:C_Small
- added C415, C416: 10uF, Capacitor_SMD:C_0603_1608Metric, symbol Device:C_Small
- added L403: 2.2uH, Inductor_SMD:L_0603_1608Metric, symbol Device:L
- added R401, R402, R403, R404: 47k, Resistor_SMD:R_0402_1005Metric, symbol Device:R_Small
- added U401: AP6212, Module_WiFi_BT:QFN-44_L12.0-W12.0-P0.90-TL_AP6212, symbol Module_WiFi_BT:AP6212
- added Y401: 26Mhz, Crystal:Crystal_SMD_3225-4Pin_3.2x2.5mm, symbol Device:Crystal_GND24
- C427, C428: now not fitted; now left out of the parts list
Connections:
- net +3V3: now also R461.1; no longer R450.1, R451.1, R452.1, R453.1, R454.1, R455.1, R456.1, R458.2, R461.2
- net ANT_FILT: now also U401.2 (WL_BT_ANT)
- net AP_WAKE_BT: now also U401.6 (BT_WAKE)
- net BT_EN: now also U401.34 (BT_RST_N)
- net BT_WAKE_AP: now also U401.7 (BT_HOST_WAKE)
- net GND: now also C402.2, C414.2, C415.2, C416.2, U401.1 (GND), U401.20 (GND), U401.3 (GND), U401.31 (GND), U401.33 (GND), U401.36 (GND), Y401.2, Y401.4
- net HCI_CTS: now also R401.2, U401.41 (UART_RTS_N)
- net HCI_RTS: now also R404.1, U401.44 (UART_CTS_N)
- net HCI_RX: now also R402.2, U401.42 (UART_TXD)
- net HCI_TX: now also R403.2, U401.43 (UART_RXD)
- net SDIO_CLK: now also U401.17 (SDIO_DATA_CLK)
- net SDIO_CMD: now also U401.16 (SDIO_DATA_CMD)
- net SDIO_D0: now also U401.18 (SDIO_DATA_0)
- net SDIO_D1: now also U401.19 (SDIO_DATA_1)
- net SDIO_D2: now also U401.14 (SDIO_DATA_2)
- net SDIO_D3: now also U401.15 (SDIO_DATA_3)
- net VDD_WIFI: now also R450.1, R451.1, R452.1, R453.1, R454.1, R455.1, R456.1, R458.2, R461.2, C415.1, C416.1, R401.1, R402.1, R403.1, R404.2, U401.22 (VDDIO), U401.9 (VBAT); no longer C429.1, R461.1
- net WL_REG_ON: now also U401.12 (WL_REG_ON)
- net WL_WAKE_AP: now also U401.13 (WL_HOST_WAKE)
- net LPO: now reaches R457.2, R458.1
- net LPO: now also U401.24 (LPO)
- new net: L403.2, U401.21 (VIN_LDO_OUT)
- new net VIN_LDO: C429.1, L403.1, U401.23 (VIN_LDO)
- new net XI: C402.1, U401.10 (XTAL_IN), Y401.1
- new net XO: C414.1, U401.11 (XTAL_OUT), Y401.3
- no-connect marks 20 -> 18
Other:
- note added: "CX1 = CX2 = 2(15pF - 2pF) = 26pF 22pF already in the bom"
- note removed: "The Datasheet calls pin 41 a ground"
- moved on the sheet: ANT401, C429, L405, R450, R451, R452, R453, R454, R455, R456, R457, R458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

Commit message: Submit for production
Signed-off-by: Connor Rigby <connorr@hey.com>
Parts:
- removed L405: 0R, Resistor_SMD:R_0402_1005Metric, symbol Device:L_Small
- added R405: 0R, Resistor_SMD:R_0402_1005Metric, symbol Device:R_Small
- C402, C414, C429, R401, R402, R403, R404, Y401: now not fitted; now left out of the parts list
- L403: LCSC C17168 -> C365953; MPN 0402WGF0000TCE -> CPY160808T-2R2M-NP; now not fitted; now left out of the parts list
- U401: value AP6212 -> RL-SM02BD-8723BS; AP6212 (none) -> C2798300; LCSC C2798300 -> C9900101851; MPN (none) -> RL-SM02BD-8723BS
Connections:
- net ANT: now also R405.1
- net ANT_FILT: now also R405.2
- net HCI_CTS renamed BT_HCI_RTS
- net HCI_RTS renamed BT_HCI_CTS
- net HCI_RX renamed BT_HCI_TX
- net HCI_TX renamed BT_HCI_RX
Changed lines of the file:
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@@
 		)
 	)
-	(hierarchical_label "HCI_CTS"
+	(hierarchical_label "BT_HCI_RTS"
 		(shape input)
 		(at 203.2 57.15 0)
@@
 		)
 	)
-	(hierarchical_label "HCI_RTS"
+	(hierarchical_label "BT_HCI_CTS"
 		(shape output)
 		(at 203.2 49.53 0)
@@
 		)
 	)
-	(hierarchical_label "HCI_TX"
+	(hierarchical_label "BT_HCI_RX"
 		(shape output)
 		(at 203.2 52.07 0)
@@
 		)
 	)
-	(hierarchical_label "HCI_RX"
+	(hierarchical_label "BT_HCI_TX"
 		(shape input)
 		(at 203.2 54.61 0)
@@
 		(unit 1)
 		(exclude_from_sim no)
-		(in_bom yes)
+		(in_bom no)
 		(on_board yes)
-		(dnp no)
+		(dnp yes)
 		(fields_autoplaced yes)
 		(property "Reference" "C414"
@@
 		(unit 1)
 		(exclude_from_sim no)
-		(in_bom yes)
+		(in_bom no)
 		(on_board yes)
-		(dnp no)
+		(dnp yes)
 		(fields_autoplaced yes)
 		(property "Reference" "R402"
@@
 		(unit 1)
 		(exclude_from_sim no)
-		(in_bom yes)
+		(in_bom no)
 		(on_board yes)
-		(dnp no)
+		(dnp yes)
 		(fields_autoplaced yes)
 		(property "Reference" "C429"
@@
 		(unit 1)
 		(exclude_from_sim no)
-		(in_bom yes)
+		(in_bom no)
 		(on_board yes)
-		(dnp no)
+		(dnp yes)
 		(property "Reference" "Y401"
 			(at 45.72 68.834 0)
@@
 	(symbol
 		(lib_id "Device:R_Small")
+		(at 55.88 43.18 90)
+		(mirror x)
+		(unit 1)
+		(exclude_from_sim no)
+		(in_bom yes)
+		(on_board yes)
+		(dnp no)
+		(fields_autoplaced yes)
+		(property "Reference" "R405"
+			(at 55.88 38.1 90)
+			(effects
+				(font
+					(size 1.27 1.27)
+				)
+			)
+		)
+		(property "Value" "0R"
+			(at 55.88 40.64 90)
+			(effects
+				(font
+					(size 1.27 1.27)
+				)
+			)
+		)
+		(property "Footprint" "Resistor_SMD:R_0402_1005Metric"
+			(at 55.88 43.18 0)
+			(effects
+				(font
+					(size 1.27 1.27)
+				)
+				(hide yes)
+			)
+		)
+		(property "Datasheet" "https://datasheet.lcsc.com/lcsc/2206010216_UNI-ROYAL-Uniroyal-Elec-0402WGF0000TCE_C17168.pdf"
+			(at 55.88 43.18 0)
+			(effects
+				(font
+					(size 1.27 1.27)
+				)
+				(hide yes)
+			)
+		)
+		(property "Description" "Resistor, small symbol"
+			(at 55.88 43.18 0)
+			(effects
+				(font
+					(size 1.27 1.27)
+				)
+				(hide yes)
+			)
+		)
+		(property "Color" ""
+			(at 55.88 43.18 0)
+			(effects
+				(font
+					(size 1.27 1.27)
+				)
+				(hide yes)
+			)
+		)
+		(property "DNP" ""
+			(at 55.88 43.18 0)
+			(effects
+				(font
+					(size 1.27 1.27)
+				)
+				(hide yes)
+			)
+		)
+		(property "LCSC" "C17168"
+			(at 55.88 43.18 0)
+			(effects
+				(font
+					(size 1.27 1.27)
+				)
+				(hide yes)
+			)
+		)
+		(property "Resistance" ""
+			(at 55.88 43.18 0)
+			(effects
+				(font
+					(size 1.27 1.27)
+				)
+				(hide yes)
+			)
+		)
+		(property "MPN" "0402WGF0000TCE"
+			(at 55.88 43.18 0)
+			(effects
+				(font
+					(size 1.27 1.27)
+				)
+				(hide yes)
+			)
+		)
+		(pin "1"
+		)
+		(pin "2"
+		)
+		(instances
+			(project "underglow3"
+				(path "/91403281-71b7-415e-b94d-23418044aa4d/ee67ecdb-9863-4cb7-8d00-48e2e9dc78dd"
+					(reference "R405")
+					(unit 1)
+				)
+			)
+		)
+	)
+	(symbol
+		(lib_id "Device:R_Small")
 		(at 87.63 135.89 0)
 		(unit 1)
@@
 			)
 		)
-		(property "Value" "AP6212"
+		(property "Value" "RL-SM02BD-8723BS"
 			(at 127 36.83 0)
 			(effects
@@
 			)
 		)
-		(property "LCSC" "C2798300"
+		(property "AP6212" "C2798300"
+			(at 127 71.12 0)
+			(effects
+				(font
+					(size 1.27 1.27)
+				)
+				(hide yes)
+			)
+		)
+		(property "LCSC" "C9900101851"
+			(at 127 71.12 0)
+			(effects
+				(font
+					(size 1.27 1.27)
+				)
+				(hide yes)
+			)
+		)
+		(property "MPN" "RL-SM02BD-8723BS"
 			(at 127 71.12 0)
 			(effects
@@
 	)
 	(symbol
-		(lib_id "Device:L_Small")
-		(at 55.88 43.18 90)
-		(unit 1)
-		(exclude_from_sim no)
-		(in_bom yes)
-		(on_board yes)
-		(dnp no)
-		(property "Reference" "L405"
-			(at 55.626 45.974 90)
-			(effects
-				(font
-					(size 1.27 1.27)
-				)
-			)
-		)
-		(property "Value" "0R"
-			(at 55.626 48.514 90)
-			(effects
-				(font
-					(size 1.27 1.27)
-				)
-			)
-		)
-		(property "Footprint" "Resistor_SMD:R_0402_1005Metric"
-			(at 55.88 43.18 0)
-			(effects
-				(font
-					(size 1.27 1.27)
-				)
-				(hide yes)
-			)
-		)
-		(property "Datasheet" "https://datasheet.lcsc.com/lcsc/2206010216_UNI-ROYAL-Uniroyal-Elec-0402WGF0000TCE_C17168.pdf"
-			(at 55.88 43.18 0)
-			(effects
-				(font
-					(size 1.27 1.27)
-				)
-				(hide yes)
-			)
-		)
-		(property "Description" "Inductor, small symbol"
-			(at 55.88 43.18 0)
-			(effects
-				(font
-					(size 1.27 1.27)
-				)
-				(hide yes)
-			)
-		)
-		(property "Color" ""
-			(at 55.88 43.18 0)
-			(effects
-				(font
-					(size 1.27 1.27)
-				)
-				(hide yes)
-			)
-		)
-		(property "DNP" ""
-			(at 55.88 43.18 0)
-			(effects
-				(font
-					(size 1.27 1.27)
-				)
-				(hide yes)
-			)
-		)
-		(property "Resistance" ""
-			(at 55.88 43.18 0)
-			(effects
-				(font
-					(size 1.27 1.27)
-				)
-				(hide yes)
-			)
-		)
-		(property "LCSC" "C17168"
-			(at 55.88 43.18 0)
-			(effects
-				(font
-					(size 1.27 1.27)
-				)
-				(hide yes)
-			)
-		)
-		(property "MPN" "0402WGF0000TCE"
-			(at 55.88 43.18 0)
-			(effects
-				(font
-					(size 1.27 1.27)
-				)
-				(hide yes)
-			)
-		)
-		(pin "2"
-		)
-		(pin "1"
-		)
-		(instances
-			(project "underglow3"
-				(path "/91403281-71b7-415e-b94d-23418044aa4d/ee67ecdb-9863-4cb7-8d00-48e2e9dc78dd"
-					(reference "L405")
-					(unit 1)
-				)
-			)
-		)
-	)
-	(symbol
 		(lib_id "Device:R_Small")
 		(at 60.96 135.89 0)
@@
 		(unit 1)
 		(exclude_from_sim no)
-		(in_bom yes)
+		(in_bom no)
 		(on_board yes)
-		(dnp no)
+		(dnp yes)
 		(fields_autoplaced yes)
 		(property "Reference" "R403"
@@
 		(unit 1)
 		(exclude_from_sim no)
-		(in_bom yes)
+		(in_bom no)
 		(on_board yes)
-		(dnp no)
+		(dnp yes)
 		(fields_autoplaced yes)
 		(property "Reference" "R401"
@@
 		(unit 1)
 		(exclude_from_sim no)
-		(in_bom yes)
+		(in_bom no)
 		(on_board yes)
-		(dnp no)
+		(dnp yes)
 		(property "Reference" "L403"
 			(at 64.77 101.6 90)
@@
 			)
 		)
-		(property "LCSC" "C17168"
+		(property "LCSC" "C365953"
 			(at 69.85 101.6 90)
 			(effects
@@
 			)
 		)
-		(property "MPN" "0402WGF0000TCE"
+		(property "MPN" "CPY160808T-2R2M-NP"
 			(at 69.85 101.6 0)
 			(effects
@@
 		(unit 1)
 		(exclude_from_sim no)
-		(in_bom yes)
+		(in_bom no)
 		(on_board yes)
-		(dnp no)
+		(dnp yes)
 		(fields_autoplaced yes)
 		(property "Reference" "C402"
@@
 		(unit 1)
 		(exclude_from_sim no)
-		(in_bom yes)
+		(in_bom no)
 		(on_board yes)
-		(dnp no)
+		(dnp yes)
 		(fields_autoplaced yes)
 		(property "Reference" "R404"
