File: MainBoard/T113-S3.kicad_sch (KiCad schematic)
At the start: 70 parts, among them J202 TC2030-IDC, J203 Micro_SD_Card_Det1, U1 T113-S3, U202 W25Q32JVSS, U203 ATECC608A-MAHDA, Y201 24Mhz

Commit message: Submit for fab rev 2
Signed-off-by: Connor Rigby <connorr@hey.com>
Parts:
- removed C206, C209, C210, C223, C226: 100nf, Capacitor_SMD:C_0402_1005Metric, symbol Device:C_Small
- removed C207, C208: 470nF, Resistor_SMD:R_0402_1005Metric, symbol Device:C_Small
- removed C224: 2.2uF, Resistor_SMD:R_0402_1005Metric, symbol Device:C_Small
- removed C225: 1nF, Resistor_SMD:R_0402_1005Metric, symbol Device:C_Small
- removed R208, R209: 22R, Resistor_SMD:R_0402_1005Metric, symbol Device:R_Small
- removed R212: 100k, Resistor_SMD:R_0402_1005Metric, symbol Device:R
- removed R215: 0R, Resistor_SMD:R_0402_1005Metric, symbol Device:R_Small
- added TP201: TVIN, TestPoint:TestPoint_Pad_D1.0mm, symbol Connector:TestPoint
- added TP202: LDOA_OUT, TestPoint:TestPoint_Pad_D1.0mm, symbol Connector:TestPoint
Connections:
- net GND: now also J203.10 (SHIELD), J203.11 (SHIELD), J203.12 (SHIELD), J203.13 (SHIELD)
- net LDOA_OUT: now also TP202.1
- net USB1_DN: now also U1.113 (USB1-DM); no longer U1.112 (USB1-DP)
- net USB1_DP: now also U1.112 (USB1-DP); no longer U1.113 (USB1-DM)
- net RELAY_COIL_VDC: now reaches U1.37 (PE10)
- net RELAY_COIL_GND: now reaches U1.38 (PE9)
- net RELAY_SW: now reaches U1.39 (PE8)
- net USB_SW: now reaches U1.84 (PB4)
- net GPADC0: no longer names the net of U1.101 (GPADC0)
- net HPOUFB: no longer names the net of U1.100 (HPOUTFB)
- net HPOUTL: no longer names the net of U1.99 (HPOUTL)
- net HPOUTR: no longer names the net of U1.98 (HPOUTR)
- net HPVCC: no longer names the net of U1.97 (HPVCC)
- net PWM5: no longer names the net of U1.53 (PD21)
- net VCC_TVIN: no longer names the net of U1.107 (VCC-TVIN)
- net VCC_TVIN: now also TP201.1
- net VRA1: no longer names the net of U1.92 (VRA1)
- net VRA2: no longer names the net of U1.90 (VRA2)
- no-connect marks 50 -> 53
Other:
- moved on the sheet: C233, J202, R213, R214, R216, TP215, TP216, TP219

Commit message: Submit for production
Signed-off-by: Connor Rigby <connorr@hey.com>
Parts:
- removed TP201: TVIN, TestPoint:TestPoint_Pad_D1.0mm, symbol Connector:TestPoint
- added D201, D202: LED, LED_SMD:LED_0402_1005Metric, symbol Device:LED
- added R208: 100k, Resistor_SMD:R_0402_1005Metric, symbol Device:R
- added R209, R212: 1k, Resistor_SMD:R_0402_1005Metric, symbol Device:R_Small
- C202, U202: now not fitted; now left out of the parts list
- J202: MPN (none) -> TC2030-IDC; now left out of the parts list
- R217, R218: LCSC C4190 -> C25879; MPN 0603WAF2201T5E -> 0402WGF2201TCE
Connections:
- net +3V3: now also D201.2 (A), D202.2 (A), R208.1
- net SPI0_CS0: now also R208.2
- net LED_ST1: now reaches U1.62 (PD7)
- net LED_ST1: now also R209.1
- net LED_ST2: now reaches U1.63 (PD8)
- net LED_ST2: now also R212.1
- new net: D202.1 (K), R212.2
- new net: D201.1 (K), R209.2
- no-connect marks 53 -> 52
