File: MainBoard/underglow3.kicad_sch (KiCad schematic)
At the start: 0 parts

Commit message: Submit for fab rev 2
Signed-off-by: Connor Rigby <connorr@hey.com>
Other:
- sheet Application ports: added RELAY_COIL_GND, RELAY_COIL_VDC, RELAY_SW, USB_SW; removed PWM5
- sheet Power ports: added RELAY_COIL_GND, RELAY_COIL_VDC, USB_SW; removed none

Commit message: Submit for production
Signed-off-by: Connor Rigby <connorr@hey.com>
Other:
- sheet RL-SM02BD-8723BS ports: added BT_HCI_CTS, BT_HCI_RTS, BT_HCI_RX, BT_HCI_TX; removed HCI_CTS, HCI_RTS, HCI_RX, HCI_TX
Changed lines of the file:
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@@
-			)
-		)
-		(pin "HCI_RTS" output
-			(at 114.3 53.34 180)
-			(effects
-				(font
-					(size 1.27 1.27)
-				)
-				(justify left)
 			)
 		)
@@
 		(pin "SDIO_CMD" input
 			(at 114.3 29.21 180)
-			(effects
-				(font
-					(size 1.27 1.27)
-				)
-				(justify left)
-			)
-		)
-		(pin "HCI_TX" output
-			(at 114.3 48.26 180)
-			(effects
-				(font
-					(size 1.27 1.27)
-				)
-				(justify left)
-			)
-		)
-		(pin "HCI_RX" input
-			(at 114.3 45.72 180)
-			(effects
-				(font
-					(size 1.27 1.27)
-				)
-				(justify left)
-			)
-		)
-		(pin "HCI_CTS" input
-			(at 114.3 50.8 180)
 			(effects
 				(font
@@
 			(effects
 				(font
+					(size 1.27 1.27)
+				)
+				(justify left)
+			)
+		)
+		(pin "BT_HCI_RTS" input
+			(at 114.3 53.34 180)
+			(effects
+				(font
+					(size 1.27 1.27)
+				)
+				(justify left)
+			)
+		)
+		(pin "BT_HCI_TX" input
+			(at 114.3 48.26 180)
+			(effects
+				(font
+					(size 1.27 1.27)
+				)
+				(justify left)
+			)
+		)
+		(pin "BT_HCI_RX" output
+			(at 114.3 45.72 180)
+			(effects
+				(font
+					(size 1.27 1.27)
+				)
+				(justify left)
+			)
+		)
+		(pin "BT_HCI_CTS" output
+			(at 114.3 50.8 180)
+			(effects
+				(font
