File: MainBoard/underglow3.kicad_pcb (KiCad board)
At the start: 4 copper layers, 81.2 x 100.2 mm, 227 parts, among them J202 TC2030-IDC, J203 Micro_SD_Card_Det1, J301 Delphi_Sicma_24, J302 USB_A, J404 USB_B_Mini, K301 G6K-2F-Y DC12, Q301 S8550, Q302 S8550, Q303 S8550, Q304 S8550, Q305 S8550, Q306 S8550, Q307 S8550, Q308 S8550, Q309 SI2302-TP, Q310 SI2302-TP, Q311 SI2302-TP, Q312 S8550, Q313 S8550, Q314 S8550, Q315 S8550, Q316 S8550, Q317 S8550, Q318 S8550, Q319 SI2302-TP, Q320 SI2302-TP, Q321 SI2302-TP, Q322 SI2301CDS-T1-GE3, U201 T113-S3, U202 W25Q32JVSS, U203 ATECC608A-MAHDA, U301 SCT2650STER, U302 USBLC6-2SC6, U303 USBLC6-2SC6, U401 RTL8723BS(ComboModule), U402 SY8088IAAC, U403 SY8088IAAC, U405 SN65HVD230, Y201 24Mhz

Commit message: Submit for fab rev 2
Signed-off-by: Connor Rigby <connorr@hey.com>
Parts:
- removed C206, C209, C210, C223, C226, C417: 100nf, Capacitor_SMD:C_0402_1005Metric
- removed C207, C208: 470nF, Resistor_SMD:R_0402_1005Metric
- removed C224: 2.2uF, Resistor_SMD:R_0402_1005Metric
- removed C225: 1nF, Resistor_SMD:R_0402_1005Metric
- removed C401: 1uF, Resistor_SMD:R_0402_1005Metric
- removed Q313, Q314, Q315, Q316, Q317, Q318: S8550, Package_TO_SOT_SMD:SOT-23
- removed Q322: SI2301CDS-T1-GE3, Package_TO_SOT_SMD:SOT-23
- removed R208, R209: 22R, Resistor_SMD:R_0402_1005Metric
- removed R212: 100k, Resistor_SMD:R_0402_1005Metric
- removed R215, R459: 0R, Resistor_SMD:R_0402_1005Metric
- added C316: 10uF, Capacitor_SMD:C_0603_1608Metric, F.Cu at (134.2, 143.4)
- added C317: 100nf, Capacitor_SMD:C_0402_1005Metric, F.Cu at (117.4, 144.8)
- added C318: 10uF, Capacitor_SMD:C_0603_1608Metric, F.Cu at (98.3, 143.4)
- added C319: 100nf, Capacitor_SMD:C_0402_1005Metric, F.Cu at (123.4, 144.8)
- added C321: 100nf, Capacitor_SMD:C_0402_1005Metric, F.Cu at (129.4, 144.8)
- added C323: 100nf, Capacitor_SMD:C_0402_1005Metric, F.Cu at (99.7, 144.9)
- added C325: 100nf, Capacitor_SMD:C_0402_1005Metric, F.Cu at (105.4, 144.8)
- added C327: 100nf, Capacitor_SMD:C_0402_1005Metric, F.Cu at (111.2, 144.8)
- added C402: 22pF, Capacitor_SMD:C_0402_1005Metric, F.Cu at (111.6, 107.5)
- added C414: 22pF, Capacitor_SMD:C_0402_1005Metric, F.Cu at (111.6, 109.5)
- added C415: 10uF, Capacitor_SMD:C_0603_1608Metric, F.Cu at (125.2, 109.3)
- added C416: 10uF, Capacitor_SMD:C_0603_1608Metric, F.Cu at (110.2, 104.7)
- added G***: LOGO, LOGO, F.Cu at (146.8, 153.7)
- added L403: 2.2uH, Inductor_SMD:L_0603_1608Metric, F.Cu at (125.2, 110.9)
- added R401: 47k, Resistor_SMD:R_0402_1005Metric, F.Cu at (119.6, 89.6)
- added R403: 47k, Resistor_SMD:R_0402_1005Metric, F.Cu at (117.3, 89.6)
- added R404: 47k, Resistor_SMD:R_0402_1005Metric, F.Cu at (116.2, 89.6)
- added TP201: TVIN, TestPoint:TestPoint_Pad_D1.0mm, F.Cu at (142.6, 106.1)
- added TP202: LDOA_OUT, TestPoint:TestPoint_Pad_D1.0mm, F.Cu at (127.3, 117.9)
- added TP301: +5V, TestPoint:TestPoint_Pad_D1.0mm, F.Cu at (81.4, 102.5)
- added TP302: gnd, TestPoint:TestPoint_Pad_D1.0mm, F.Cu at (83.4, 102.5)
- added TP303: +3.3V, TestPoint:TestPoint_Pad_D1.0mm, F.Cu at (114.2, 120.1)
- added TP304: gnd, TestPoint:TestPoint_Pad_D1.0mm, F.Cu at (114.2, 121.7)
- added U304: MCP1416T-E/OT, Package_TO_SOT_SMD:SOT-23-5, F.Cu at (119.4, 144.0)
- added U305: MCP1416T-E/OT, Package_TO_SOT_SMD:SOT-23-5, F.Cu at (125.5, 144.0)
- added U306: MCP1416T-E/OT, Package_TO_SOT_SMD:SOT-23-5, F.Cu at (131.5, 144.0)
- added U307: MCP1416T-E/OT, Package_TO_SOT_SMD:SOT-23-5, F.Cu at (101.7, 144.0)
- added U308: MCP1416T-E/OT, Package_TO_SOT_SMD:SOT-23-5, F.Cu at (107.5, 144.0)
- added U309: MCP1416T-E/OT, Package_TO_SOT_SMD:SOT-23-5, F.Cu at (113.5, 144.0)
- added Y401: 26Mhz, Crystal:Crystal_SMD_3225-4Pin_3.2x2.5mm, F.Cu at (109.3, 108.4)
- added kibuzzard-65F09D1C: G***, kibuzzard-65F09D1C, F.Cu at (130.3, 133.9)
- added kibuzzard-65FE521F: G***, kibuzzard-65FE521F, F.Cu at (79.8, 102.5)
- added kibuzzard-65FE522B: G***, kibuzzard-65FE522B, F.Cu at (85.1, 102.5)
- added kibuzzard-65FE522B: G***, kibuzzard-65FE522B, F.Cu at (115.9, 121.7)
- added kibuzzard-65FE52BD: G***, kibuzzard-65FE52BD, F.Cu at (153.8, 112.9)
- added kibuzzard-65FEF020: G***, kibuzzard-65FEF020, F.Cu at (115.9, 120.1)
- added kibuzzard-65FEF408: G***, kibuzzard-65FEF408, F.Cu at (128.9, 118.0)
- added kibuzzard-65FEF568: G***, kibuzzard-65FEF568, F.Cu at (81.6, 142.7)
- Q301, Q304, Q307: value S8550 -> AO3419; footprint Package_TO_SOT_SMD:SOT-23 -> Package_TO_SOT_SMD:SOT-23W
- Q302, Q303, Q305, Q306: value S8550 -> SI2302-TP
- Q308, Q312: value S8550 -> MMBT5551
- R306, R328: value 100k 1% -> 22R
- R316, R317, R318, R330: value 100k 1% -> 1k
- R321, R322, R331, R333, R334: value 1k -> 100k 1%
- R323, R324: value 1k -> 22R
- R402: value 1k -> 47k
- U401: value RTL8723BS(ComboModule) -> AP6212
- moved Q307 77.5 mm to (107.3, 74.5)
- moved R334 71.0 mm to (106.4, 71.9), turned to 180 degrees
- moved R402 56.9 mm to (118.5, 89.6)
- moved Q304 50.0 mm to (88.9, 149.7), turned to -90 degrees
- moved Q306 48.1 mm to (82.3, 147.4), turned to 180 degrees
- moved R321 46.6 mm to (94.6, 149.3), turned to 180 degrees
- moved R324 46.2 mm to (89.8, 152.5), turned to 180 degrees
- moved Q305 40.9 mm to (82.4, 151.5), turned to 180 degrees
- moved R323 40.7 mm to (87.8, 152.5)
- moved Q303 40.1 mm to (91.6, 151.5), turned to 180 degrees
- moved R320 38.6 mm to (94.6, 148.2), turned to 180 degrees
- moved R332 33.0 mm to (85.3, 148.4), turned to 180 degrees
- moved Q302 31.9 mm to (91.6, 147.3), turned to 180 degrees
- moved R322 31.5 mm to (88.7, 147.2), turned to 180 degrees
- moved R302 29.6 mm to (126.8, 147.4), turned to -90 degrees
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Connections:
- net Net-(U401-SUSCLK_IN/GPIO6) renamed /RL-SM02BD-8723BS/LPO
- C429 pad 1: /RL-SM02BD-8723BS/VDD_WIFI -> /RL-SM02BD-8723BS/VIN_LDO
- D305 pad 1: /Power/VIN -> Net-(D305-K)
- D408 pad 1: +5V -> Net-(D408-K)
- D408 pad 2: Net-(D408-A) -> +5V
- D409 pad 1: +3V3 -> Net-(D409-K)
- D409 pad 2: Net-(D409-A) -> +3V3
- J203 pad 10: unconnected-(J203-SHIELD-Pad10) -> GND
- J203 pad 11: unconnected-(J203-SHIELD-Pad10)_2 -> GND
- J203 pad 12: unconnected-(J203-SHIELD-Pad10)_1 -> GND
- J203 pad 13: unconnected-(J203-SHIELD-Pad10)_0 -> GND
- K301 pad 1: /Power/VIN -> Net-(D305-K)
- Q301 pad 1: Net-(Q301-B) -> Net-(Q301-G)
- Q301 pad 2: GND -> +5V
- Q301 pad 3: Net-(D305-A) -> Net-(Q301-D)
- Q302 pad 1: Net-(Q302-B) -> Net-(Q302-G)
- Q302 pad 2: Net-(Q302-E) -> GND
- Q302 pad 3: GND -> Net-(Q302-D)
- Q303 pad 1: Net-(Q303-B) -> Net-(Q302-D)
- Q303 pad 2: Net-(Q303-E) -> GND
- Q303 pad 3: GND -> Net-(Q303-D)
- Q304 pad 1: Net-(Q304-B) -> Net-(Q302-D)
- Q304 pad 2: Net-(Q304-E) -> +5V
- Q304 pad 3: GND -> Net-(Q304-D)
- Q305 pad 1: Net-(Q302-E) -> Net-(Q305-G)
- Q305 pad 2: Net-(Q305-E) -> GND
- Q305 pad 3: GND -> Net-(Q305-D)
- Q306 pad 1: Net-(Q303-E) -> Net-(Q306-G)
- Q306 pad 2: Net-(Q306-E) -> GND
- Q306 pad 3: GND -> Net-(Q301-G)
- Q307 pad 1: Net-(Q304-E) -> Net-(Q307-G)
- Q307 pad 2: Net-(Q307-E) -> +5V
- Q307 pad 3: GND -> Net-(J302-VBUS)
- Q309 pad 1: Net-(Q305-E) -> /Power/RGB1_R_G
- Q310 pad 1: Net-(Q306-E) -> /Power/RGB1_G_G
- Q311 pad 1: Net-(Q307-E) -> /Power/RGB1_B_G
- Q319 pad 1: Net-(Q316-E) -> /Power/RGB2_R_G
- Q320 pad 1: Net-(Q317-E) -> /Power/RGB2_G_G
- Q321 pad 1: Net-(Q318-E) -> /Power/RGB2_B_G
- R301 pad 1: /Power/RGB2_OUT -> Net-(U304-OUT)
- R301 pad 2: Net-(Q313-E) -> /Power/RGB1_R_G
- R302 pad 1: /Power/RGB2_OUT -> Net-(U305-OUT)
- R302 pad 2: Net-(Q316-E) -> /Power/RGB1_G_G
- R303 pad 1: Net-(Q322-G) -> Net-(Q307-G)
- R303 pad 2: /Power/USB_SW -> /Application/USB_SW
- R306 pad 1: Net-(Q301-B) -> Net-(Q301-D)
- R306 pad 2: GND -> Net-(D305-K)
- R316 pad 1: Net-(Q302-B) -> Net-(U306-OUT)
- R316 pad 2: GND -> /Power/RGB1_B_G
- R317 pad 1: Net-(Q303-B) -> Net-(U307-OUT)
- R317 pad 2: GND -> /Power/RGB2_R_G
- R318 pad 1: Net-(Q304-B) -> Net-(U308-OUT)
- R318 pad 2: GND -> /Power/RGB2_G_G
- R319 pad 1: /Power/RGB1_OUT -> Net-(U309-OUT)
- R319 pad 2: Net-(Q302-E) -> /Power/RGB2_B_G
- R320 pad 1: /Power/RGB1_OUT -> /Application/RELAY_SW
- R320 pad 2: Net-(Q303-E) -> Net-(Q302-G)
- R321 pad 1: /Power/RGB1_OUT -> /Application/RELAY_SW
- R321 pad 2: Net-(Q304-E) -> GND
- R322 pad 1: /Power/RGB1_OUT -> Net-(Q302-D)
- R322 pad 2: Net-(Q305-E) -> +5V
- R323 pad 1: /Power/RGB1_OUT -> Net-(Q304-D)
- R323 pad 2: Net-(Q306-E) -> Net-(D305-A)
- R324 pad 1: /Power/RGB1_OUT -> Net-(Q303-D)
- R324 pad 2: Net-(Q307-E) -> Net-(D305-A)
- R328 pad 1: Net-(Q313-B) -> Net-(Q305-D)
- R328 pad 2: GND -> Net-(D305-K)
- R329 pad 1: Net-(Q314-B) -> /Application/RELAY_COIL_GND
- R330 pad 1: Net-(Q315-B) -> /Application/RELAY_COIL_GND
- R330 pad 2: GND -> Net-(Q305-G)
- R331 pad 1: /Power/RGB2_OUT -> /Application/RELAY_COIL_VDC
- R331 pad 2: Net-(Q314-E) -> GND
- R332 pad 1: /Power/RGB2_OUT -> /Application/RELAY_COIL_VDC
- R332 pad 2: Net-(Q315-E) -> Net-(Q306-G)
- R333 pad 1: /Power/RGB2_OUT -> Net-(Q301-G)
- R333 pad 2: Net-(Q317-E) -> +5V
- R334 pad 1: /Power/RGB2_OUT -> Net-(Q307-G)
- R334 pad 2: Net-(Q318-E) -> GND
- R402 pad 1: /Application/PWM5 -> /RL-SM02BD-8723BS/VDD_WIFI
- R402 pad 2: Net-(Q301-B) -> /Application/HCI_TX
- R408 pad 1: Net-(Q313-B) -> Net-(U307-IN)
- R411 pad 1: Net-(Q304-B) -> Net-(U306-IN)
- R427 pad 2: Net-(D408-A) -> Net-(D408-K)
- R428 pad 2: Net-(D409-A) -> Net-(D409-K)
- R430 pad 1: Net-(Q315-B) -> Net-(U309-IN)
- R434 pad 1: Net-(Q314-B) -> Net-(U308-IN)
- R435 pad 2: Net-(Q303-B) -> Net-(U305-IN)
- R436 pad 2: Net-(Q302-B) -> Net-(U304-IN)
- R450 pad 1: +3V3 -> /RL-SM02BD-8723BS/VDD_WIFI
- R451 pad 1: +3V3 -> /RL-SM02BD-8723BS/VDD_WIFI
- R452 pad 1: +3V3 -> /RL-SM02BD-8723BS/VDD_WIFI
- R453 pad 1: +3V3 -> /RL-SM02BD-8723BS/VDD_WIFI
- R454 pad 1: +3V3 -> /RL-SM02BD-8723BS/VDD_WIFI
- R455 pad 1: +3V3 -> /RL-SM02BD-8723BS/VDD_WIFI
- R456 pad 1: +3V3 -> /RL-SM02BD-8723BS/VDD_WIFI
- R458 pad 2: +3V3 -> /RL-SM02BD-8723BS/VDD_WIFI
- R461 pad 1: /RL-SM02BD-8723BS/VDD_WIFI -> +3V3
- R461 pad 2: +3V3 -> /RL-SM02BD-8723BS/VDD_WIFI
- U201 pad 100: /Application/HPOUFB -> unconnected-(U201-HPOUTFB-Pad100)
- U201 pad 101: /Application/GPADC0 -> unconnected-(U201-GPADC0-Pad101)
- U201 pad 107: /Application/VCC_TVIN -> Net-(U201-VCC-TVIN)
- U201 pad 112: /Application/USB1_DN -> /Application/USB1_DP
- U201 pad 113: /Application/USB1_DP -> /Application/USB1_DN
- U201 pad 37: unconnected-(U201-PE10-Pad37) -> /Application/RELAY_COIL_VDC
- U201 pad 38: unconnected-(U201-PE9-Pad38) -> /Application/RELAY_COIL_GND
- U201 pad 39: unconnected-(U201-PE8-Pad39) -> /Application/RELAY_SW
- U201 pad 53: /Application/PWM5 -> unconnected-(U201-PD21-Pad53)
- U201 pad 84: unconnected-(U201-PB4-Pad84) -> /Application/USB_SW
- U201 pad 90: /Application/VRA2 -> unconnected-(U201-VRA2-Pad90)
- U201 pad 92: /Application/VRA1 -> unconnected-(U201-VRA1-Pad92)
- U201 pad 97: /Application/HPVCC -> unconnected-(U201-HPVCC-Pad97)
- U201 pad 98: /Application/HPOUTR -> unconnected-(U201-HPOUTR-Pad98)
- U201 pad 99: /Application/HPOUTL -> unconnected-(U201-HPOUTL-Pad99)
- U401 pad 10: unconnected-(U401-NC-Pad10) -> /RL-SM02BD-8723BS/XI
- U401 pad 11: unconnected-(U401-NC-Pad11) -> /RL-SM02BD-8723BS/XO
- U401 pad 21: unconnected-(U401-NC-Pad21) -> Net-(U401-VIN_LDO_OUT)
- U401 pad 23: unconnected-(U401-NC-Pad23) -> /RL-SM02BD-8723BS/VIN_LDO
- U401 pad 3: unconnected-(U401-NC-Pad3) -> GND
- U401 pad 41: /Application/HCI_CTS -> /Application/HCI_RTS
- U401 pad 42: /Application/HCI_RX -> /Application/HCI_TX
- U401 pad 43: /Application/HCI_TX -> /Application/HCI_RX
- U401 pad 44: /Application/HCI_RTS -> /Application/HCI_CTS
Routing:
- net +3V3: track 320.0 -> 240.5 mm, vias 31 -> 19
- net /Application/RELAY_SW: track 0.00 -> 77.1 mm
- net /Application/RELAY_COIL_GND: track 0.00 -> 76.6 mm
- net /Application/USB_SW: track 0.00 -> 76.6 mm
- net /Application/RELAY_COIL_VDC: track 0.00 -> 72.3 mm
- net /RL-SM02BD-8723BS/VDD_WIFI: track 28.9 -> 95.0 mm, vias 0 -> 7
- net /Application/PWM5: track 62.7 -> 0.00 mm
- net GND: track 113.8 -> 86.1 mm, vias 198 -> 221
- net /Application/LDOA_OUT: track 60.7 -> 34.4 mm, vias 2 -> 0
- net GNDA: track 28.8 -> 5.78 mm
- net Net-(D304-K): track 53.1 -> 75.6 mm
- net /Power/VIN: track 51.4 -> 37.6 mm
- net Net-(D305-K): track 0.00 -> 11.6 mm
- net Net-(Q302-D): track 0.00 -> 11.0 mm
- net /Application/LEDC: track 67.3 -> 58.5 mm, vias 2 -> 0
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- removed copper zone on B.Cu, net +3V3
Other:
- outline, holes or cut-outs redrawn

Commit message: Submit for production
Signed-off-by: Connor Rigby <connorr@hey.com>
Parts:
- removed C202: 100nf, Capacitor_SMD:C_0402_1005Metric
- removed C301: 1uF, Resistor_SMD:R_0402_1005Metric
- removed C305: 22pF, Capacitor_SMD:C_0402_1005Metric
- removed C306: 3.3nF, Capacitor_SMD:C_0402_1005Metric
- removed C308: 10uF, Capacitor_SMD:C_0603_1608Metric
- removed C309: 220nF, Capacitor_SMD:C_0603_1608Metric
- removed C310: 68pF, Capacitor_SMD:C_0603_1608Metric
- removed FB302: 450mΩ ±25% 600Ω@100MHz, Inductor_SMD:L_0603_1608Metric
- removed L301: 8.2uH 3.7A, Inductor_LCSC:IND-SMD_L7.0-W6.6_FXL0630
- removed L302: 2.2uH, Inductor_SMD:L_0603_1608Metric
- removed L405: 0R, Inductor_SMD:L_0402_1005Metric
- removed Q308, Q312: MMBT5551, Package_TO_SOT_SMD:SOT-23
- removed R304, R305: 0R, Resistor_SMD:R_0402_1005Metric
- removed R309, R310, R314: 100k 1%, Resistor_SMD:R_0402_1005Metric
- removed R313: 33k 1%, Resistor_SMD:R_0402_1005Metric
- removed R315: 18.7k 1%, Resistor_SMD:R_0402_1005Metric
- removed R446: 1k, Resistor_SMD:R_0402_1005Metric
- removed TP201: TVIN, TestPoint:TestPoint_Pad_D1.0mm
- removed U202: W25Q32JVSS, Package_SO:SOIC-8_5.23x5.23mm_P1.27mm
- removed U301: SCT2650STER, Package_SO:HSOP-8-1EP_3.9x4.9mm_P1.27mm_EP2.41x3.1mm
- removed kibuzzard-65FE521F: G***, kibuzzard-65FE521F
- removed the kibuzzard-65FE522B at (85.1, 102.5)
- added D201: LED, LED_SMD:LED_0402_1005Metric, F.Cu at (142.1, 133.5)
- added D202: LED, LED_SMD:LED_0402_1005Metric, F.Cu at (143.2, 133.5)
- added D301: LED, LED_SMD:LED_0402_1005Metric, F.Cu at (119.9, 142.0)
- added D302: LED, LED_SMD:LED_0402_1005Metric, F.Cu at (125.9, 142.0)
- added D303: LED, LED_SMD:LED_0402_1005Metric, F.Cu at (131.9, 142.0)
- added D307: LED, LED_SMD:LED_0402_1005Metric, F.Cu at (102.2, 142.0)
- added D308: LED, LED_SMD:LED_0402_1005Metric, F.Cu at (108.0, 142.0)
- added D309: LED, LED_SMD:LED_0402_1005Metric, F.Cu at (113.9, 142.0)
- added D310: LED, LED_SMD:LED_0402_1005Metric, F.Cu at (90.0, 139.6)
- added D311: LED, LED_SMD:LED_0402_1005Metric, F.Cu at (87.7, 139.6)
- added D312: LED, LED_SMD:LED_0402_1005Metric, F.Cu at (84.8, 139.6)
- added D313: NSR0320MW2T1G, Diode_SMD:D_SOD-323, F.Cu at (95.6, 139.6)
- added L303: 4.7uH, easyeda2kicad:IND-SMD_L7.3-W7.3, F.Cu at (89.2, 92.1)
- added R209: 1k, Resistor_SMD:R_0402_1005Metric, F.Cu at (142.1, 131.6)
- added R212: 1k, Resistor_SMD:R_0402_1005Metric, F.Cu at (143.2, 131.6)
- added R335: 1k, Resistor_SMD:R_0402_1005Metric, F.Cu at (117.9, 142.0)
- added R336: 1k, Resistor_SMD:R_0402_1005Metric, F.Cu at (123.9, 142.0)
- added R337: 1k, Resistor_SMD:R_0402_1005Metric, F.Cu at (129.9, 142.0)
- added R338: 1k, Resistor_SMD:R_0402_1005Metric, F.Cu at (100.2, 142.0)
- added R339: 1k, Resistor_SMD:R_0402_1005Metric, F.Cu at (106.0, 142.0)
- added R340: 1k, Resistor_SMD:R_0402_1005Metric, F.Cu at (111.7, 142.0)
- added R341: 1k, Resistor_SMD:R_0402_1005Metric, F.Cu at (89.8, 138.2)
- added R342: 1k, Resistor_SMD:R_0402_1005Metric, F.Cu at (87.2, 138.2)
- added R343: 1k, Resistor_SMD:R_0402_1005Metric, F.Cu at (85.3, 138.2)
- added R344: 100k 1%, Resistor_SMD:R_0402_1005Metric, F.Cu at (110.1, 143.6)
- added R345: 100k 1%, Resistor_SMD:R_0402_1005Metric, F.Cu at (104.4, 143.6)
- added R346: 100k 1%, Resistor_SMD:R_0402_1005Metric, F.Cu at (98.6, 143.6)
- added R347: 10k, Resistor_SMD:R_0402_1005Metric, F.Cu at (84.6, 101.3)
- added R348: 3.3k, Resistor_SMD:R_0402_1005Metric, F.Cu at (84.6, 103.3)
- added R405: 0R, Resistor_SMD:R_0402_1005Metric, F.Cu at (111.2, 97.1)
- added U310: TPS5430DDA, Package_SO:TI_SO-PowerPAD-8_ThermalVias, F.Cu at (89.1, 100.8)
- added kibuzzard-6669C582: G***, kibuzzard-6669C582, F.Cu at (82.0, 89.7)
- added kibuzzard-6669C587: G***, kibuzzard-6669C587, F.Cu at (82.0, 87.8)
- added kibuzzard-666C6B51: G***, kibuzzard-666C6B51, F.Cu at (97.1, 110.9)
- K301: value G6K-2F-Y DC12 -> G6K-2F-Y-TR DC3
- R307, R311: footprint Resistor_SMD:R_0603_1608Metric -> Resistor_SMD:R_0402_1005Metric
- R308, R312: value 2.2k -> 3.9k; footprint Resistor_SMD:R_0603_1608Metric -> Resistor_SMD:R_0402_1005Metric
- R326, R327: value 1k -> 100k 1%
- U201: footprint Package_QFP:LQFP-128_14x14mm_P0.4mm -> CPU_Allwinner_T113-S3:LQFP-128_L14.0-W14.0-P0.40-LS16.0-BL-EP5.6
- U302, U303: value USBLC6-2SC6 -> SRV05-4
- U401: value AP6212 -> RL-SM02BD-8723BS; footprint Module_WiFi_BT:RL-SM02BD(RTL8723BS) -> Module_WiFi_BT:QFN-44_L12.0-W12.0-P0.90-TL_AP6212
- moved G*** 77.4 mm to (82.4, 110.7)
- moved R327 31.8 mm to (128.3, 143.6)
- moved R326 28.5 mm to (122.3, 143.6)
- moved FB403 26.8 mm to (106.6, 83.1), turned to -90 degrees
- moved R325 24.5 mm to (116.3, 143.6), turned to -90 degrees
- moved D405 23.9 mm to (104.0, 82.3), turned to 180 degrees
- moved R203 21.3 mm to (125.8, 115.2)
- moved TP302 14.7 mm to (83.8, 87.8), turned to 180 degrees
- moved TP303 13.7 mm to (102.6, 127.3)
- moved kibuzzard-65FEF020 13.7 mm to (104.3, 127.3)
- moved TP304 13.7 mm to (102.6, 128.9)
- moved kibuzzard-65FE522B 13.7 mm to (104.3, 128.9)
- moved TP301 13.0 mm to (83.8, 89.7), turned to 180 degrees
- moved D306 11.7 mm to (94.8, 100.7), turned to -90 degrees
- moved R206 9.97 mm to (125.8, 116.2), turned to 180 degrees
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Connections:
- net /Power/SW renamed /Power/PH
- C304 pad 1: Net-(U301-BOOT) -> /Power/BOOT
- C311 pad 1: Net-(C311-Pad1) -> +5V
- C313 pad 1: Net-(C308-Pad1) -> +5V
- C314 pad 1: Net-(C308-Pad1) -> +5V
- J302 pad 2: Net-(J302-D-) -> /Power/USB1_DN
- J302 pad 3: Net-(J302-D+) -> /Power/USB1_DP
- J302 pad 6: (no net) -> unconnected-(J302-Shield-Pad5)
- J404 pad 2: Net-(J404-D-) -> /Power/USB0_DN
- J404 pad 3: Net-(J404-D+) -> /Power/USB0_DP
- R325 pad 1: Net-(Q308-B) -> GND
- R325 pad 2: GND -> Net-(U304-IN)
- R326 pad 1: +5V -> GND
- R326 pad 2: Net-(Q308-E) -> Net-(U305-IN)
- R327 pad 1: +5V -> GND
- R327 pad 2: /Power/LEDC_OUT -> Net-(U306-IN)
- R401 pad 2: /Application/HCI_RTS -> /Application/HCI_CTS
- R402 pad 2: /Application/HCI_TX -> /Application/HCI_RX
- R403 pad 2: /Application/HCI_RX -> /Application/HCI_TX
- R404 pad 1: /Application/HCI_CTS -> /Application/HCI_RTS
- TP301 pad 1: Net-(C308-Pad1) -> +5V
- U201 pad 107: Net-(U201-VCC-TVIN) -> unconnected-(U201-VCC-TVIN-Pad107)
- U201 pad 112: /Application/USB1_DP -> /Power/USB1_DP
- U201 pad 113: /Application/USB1_DN -> /Power/USB1_DN
- U201 pad 114: /Application/USB0_DN -> /Power/USB0_DN
- U201 pad 115: /Application/USB0_DP -> /Power/USB0_DP
- U201 pad 62: unconnected-(U201-PD7-Pad62) -> /Application/LED_ST1
- U201 pad 63: unconnected-(U201-PD8-Pad63) -> /Application/LED_ST2
- U302 pad 1: Net-(J302-D-) -> /Power/USB1_DN
- U302 pad 3: Net-(J302-D+) -> /Power/USB1_DP
- U302 pad 4: /Application/USB1_DP -> /Power/USB1_DP
- U302 pad 6: /Application/USB1_DN -> /Power/USB1_DN
- U303 pad 1: Net-(J404-D-) -> /Power/USB0_DN
- U303 pad 3: Net-(J404-D+) -> /Power/USB0_DP
- U303 pad 4: /Application/USB0_DP -> /Power/USB0_DP
- U303 pad 6: /Application/USB0_DN -> /Power/USB0_DN
- U401 pad 41: /Application/HCI_RTS -> /Application/HCI_CTS
- U401 pad 42: /Application/HCI_TX -> /Application/HCI_RX
- U401 pad 43: /Application/HCI_RX -> /Application/HCI_TX
- U401 pad 44: /Application/HCI_CTS -> /Application/HCI_RTS
Routing:
- net /Power/USB0_DP: track 0.00 -> 71.8 mm
- net /Power/USB0_DN: track 0.00 -> 70.2 mm
- net /Application/USB0_DP: track 68.1 -> 0.00 mm
- net /Power/USB1_DP: track 0.00 -> 67.8 mm
- net /Application/USB0_DN: track 66.3 -> 0.00 mm
- net /Application/USB1_DP: track 65.9 -> 0.00 mm
- net /Power/USB1_DN: track 0.00 -> 65.7 mm
- net /Application/USB1_DN: track 63.4 -> 0.00 mm
- net GND: track 86.1 -> 36.0 mm, vias 221 -> 197
- net +5V: track 192.6 -> 229.4 mm, vias 7 -> 18
- net /Power/VBUS: track 38.5 -> 2.81 mm
- net /Application/SPI0_CLK: track 34.5 -> 0.00 mm, vias 2 -> 0
- net /Application/SPI0_WP: track 34.3 -> 0.00 mm, vias 2 -> 0
- net /Application/SPI0_CS0: track 34.0 -> 0.00 mm, vias 2 -> 0
- net /Application/SPI0_HLD: track 32.4 -> 0.00 mm, vias 2 -> 0
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- added copper zone on F.Cu, net +5V
- added copper zone on F.Cu, net /Power/VBUS
- removed copper zone on F.Cu, net Net-(C308-Pad1)
Other:
- outline, holes or cut-outs redrawn

Commit message: Doc updates
Signed-off-by: Connor Rigby <connorr@hey.com>
Routing:
- net /Power/VIN: track 37.2 -> 36.7 mm
Changed lines of the file:
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@@
 			(pintype "passive+no_connect")
 		)
-		(model "C:/Users/konno/Desktop/workspace/connorrigby/underglow3/library/work/JLC2KiCad_lib/footprint/packages3d/USB-A-SMD_USB-234-BCW.step"
+		(model "${KIPRJMOD}/../library/work/JLC2KiCad_lib/footprint/packages3d/USB-A-SMD_USB-234-BCW.step"
 			(offset
 				(xyz 0 -5.000066 4.000001)
@@
 			)
 		)
-		(model "C:/Users/konno/Desktop/workspace/connorrigby/underglow3/library/Connector_LCSC_USB.pretty/packages3d/mini_usb_wifi_adapter.stp"
+		(model "${KIPRJMOD}/../library/Connector_LCSC_USB.pretty/packages3d/mini_usb_wifi_adapter.stp"
 			(offset
 				(xyz 0 -15 4)
@@
 	)
 	(segment
-		(start 86.2 160.270254)
-		(end 79.1 160.270254)
-		(width 1)
+		(start 103 165.870254)
+		(end 92.2 165.870254)
+		(width 2)
 		(layer "F.Cu")
 		(net 34)
 	)
 	(segment
-		(start 103 165.870254)
-		(end 92.2 165.870254)
-		(width 2)
+		(start 86.2 160.270254)
+		(end 79.6 160.270254)
+		(width 1)
 		(layer "F.Cu")
 		(net 34)
@@
 	(segment
 		(start 86.2 166.220254)
+		(end 86.2 160.270254)
+		(width 1)
+		(layer "F.Cu")
+		(net 34)
+	)
+	(segment
+		(start 86.2 166.220254)
 		(end 82.4775 166.220254)
 		(width 1)
@@
 		(width 1)
 		(layer "F.Cu")
-		(net 34)
-	)
-	(segment
-		(start 86.2 166.220254)
-		(end 86.2 160.270254)
-		(width 1)
-		(layer "F.Cu")
